Commit message: scripts

File: src/bluerov_simulation_blackbox/urdf/urdf.xacro (robot description, xacro)
@@ -4,5 +4,5 @@
     <link name="bluerov2/base_link">
       <inertial>
-        <origin rpy="3.1416 0 1.57" xyz="0.0 0.0 0.011" />
+        <origin rpy="3.1416 0 0" xyz="0.0 0.0 0.011" />
         <mass value="13.0" />
         <inertia
@@ -22,5 +22,5 @@
           />
         </geometry>
-        <origin rpy="3.1416 0 1.57" xyz="0 0 0" />
+        <origin rpy="3.1416 0 0" xyz="0 0 0" />
       </visual>
       <collision name="base_link_collision">
@@ -28,5 +28,5 @@
           <box size="0.457 0.575 0.05" />
         </geometry>
-        <origin rpy="3.1416 0 1.57" xyz="0 0 0.06" />
+        <origin rpy="3.1416 0 0" xyz="0 0 0.06" />
       </collision>
     </link>
@@ -34,5 +34,5 @@
     <xacro:include filename="$(find bluerov_simulation_blackbox)/urdf/description/camera/urdf.xacro" />
     <xacro:camera_urdf prefix="" parent="bluerov2/base_link">
-      <origin rpy="0 0 0" xyz="0.0 0.18 -0.06" />
+      <origin rpy="0 0 -1.57" xyz="0.18 0.0 -0.06" />
     </xacro:camera_urdf>
     <!-- Import T200 macro -->
